Commit message: mecanum

File: src/mecanum_description/urdf/mecanum.urdf.xacro (robot description, xacro)
@@ -12,4 +12,7 @@
   <!-- Include ros2_control Plugins -->
   <xacro:include filename="$(find mecanum_description)/urdf/mecanum_ros2_control.xacro" />
+    <xacro:property name="wheel_radius" value="0.075" />
+  <xacro:property name="wheel_width" value="0.045" />
+  <xacro:property name="PI" value="3.1415926535897931" />
   <link
     name="base_link">
@@ -83,10 +86,6 @@
     </visual>
     <collision>
-      <origin
-        xyz="0 0 0"
-        rpy="0 0 0" />
-      <geometry>
-        <mesh
-          filename="package://mecanum_description/meshes/Wheel_fl.STL" />
+      <geometry>
+        <sphere radius="${wheel_radius}"/>
       </geometry>
     </collision>
@@ -136,10 +135,6 @@
     </visual>
     <collision>
-      <origin
-        xyz="0 0 0"
-        rpy="0 0 0" />
-      <geometry>
-        <mesh
-          filename="package://mecanum_description/meshes/Wheel_fr.STL" />
+      <geometry>
+        <sphere radius="${wheel_radius}"/>
       </geometry>
     </collision>
@@ -156,5 +151,5 @@
       link="Wheel_fr" />
     <axis
-      xyz="0 -1 0" />
+      xyz="0 1 0" />
   </joint>
   <link
@@ -189,10 +184,6 @@
     </visual>
     <collision>
-      <origin
-        xyz="0 0 0"
-        rpy="0 0 0" />
-      <geometry>
-        <mesh
-          filename="package://mecanum_description/meshes/Wheel_rl.STL" />
+      <geometry>
+        <sphere radius="${wheel_radius}"/>
       </geometry>
     </collision>
@@ -242,10 +233,6 @@
     </visual>
     <collision>
-      <origin
-        xyz="0 0 0"
-        rpy="0 0 0" />
-      <geometry>
-        <mesh
-          filename="package://mecanum_description/meshes/Wheel_rr.STL" />
+      <geometry>
+        <sphere radius="${wheel_radius}"/>
       </geometry>
     </collision>
